File: 4-port PSE.kicad_pcb (KiCad board)
At the start: 2 copper layers, 69.8 x 54.6 mm, 23 parts, among them J1 1x7 2.54mm PV Female Header, U1 MP3924GU-Z

Commit message: V2.0 - ESP32-C6 controlled
Parts:
- added BOOT: TS-1088-AR02016, TS-1088-AR02016:SW_TS-1088_XNP, F.Cu at (106.3, 42.3)
- added C1: 22µF, Capacitor_SMD:C_0603_1608Metric, F.Cu at (120.2, 40.6)
- added C2: 0.1µF, Capacitor_SMD:C_0603_1608Metric, F.Cu at (118.2, 40.6)
- added J2: GT-USB-7004, GT-USB-7004:CONN12_B-7004_GSW, F.Cu at (135.8, 65.8)
- added R1: 4.7kΩ, ±1%, Resistor_SMD:R_0603_1608Metric, F.Cu at (133.7, 65.5)
- added R2: 4.7kΩ, ±1%, Resistor_SMD:R_0603_1608Metric, F.Cu at (133.7, 60.7)
- added R3: 4.7kΩ, ±1%, Resistor_SMD:R_0603_1608Metric, F.Cu at (113.9, 50.5)
- added R4: 4.7kΩ, ±1%, Resistor_SMD:R_0603_1608Metric, F.Cu at (113.9, 48.0)
- added R5: 4.7kΩ, ±1%, Resistor_SMD:R_0603_1608Metric, F.Cu at (122.3, 41.6)
- added RESET: TS-1088-AR02016, TS-1088-AR02016:SW_TS-1088_XNP, F.Cu at (113.8, 42.3)
- added U2: ESP32-C6-WROOM-1-N8, ESP32-C6-WROOM-1:MOD28_ESP32-C6-WROOM-1_EXP, F.Cu at (133.0, 44.8)
- C_PORT1, C_PORT2, C_PORT3, C_PORT4, C_VIN2: value 0.1µF, 100V -> 0.1µF; footprint ThickSilk:C_1206_3216Metric -> Capacitor_SMD:C_0805_2012Metric
- C_VIN1: value 220µF, 100V -> 220µF
- R_EN: footprint Resistor_SMD:R_0402_1005Metric -> Resistor_SMD:R_0603_1608Metric
- R_PMAX: footprint Resistor_SMD:R_1206_3216Metric -> Resistor_SMD:R_0805_2012Metric
- R_SENSE1, R_SENSE2, R_SENSE3, R_SENSE4: value 250mΩ, ±1% -> 250mΩ, ±1%, 100V
- ZD_PORT1, ZD_PORT2, ZD_PORT3, ZD_PORT4: value SMBJ58A -> 58V Vrwm, 95V Vc; footprint ThickSilk:D_SMB -> Diode_SMD:D_SMB
- moved R_EN 0.36 mm to (105.3, 47.0)
- moved C_PORT1 0.25 mm to (126.9, 77.6)
- moved C_PORT2 0.25 mm to (111.9, 77.6)
- moved C_PORT3 0.25 mm to (93.0, 77.6)
- moved C_VIN2 0.25 mm to (92.8, 47.7)
- moved R_PMAX 0.25 mm to (96.4, 47.7)
- moved C_PORT4 0.25 mm to (77.9, 77.3)
- moved ZD_PORT2 0.25 mm to (111.9, 73.7)
- moved ZD_PORT3 0.25 mm to (93.0, 73.7)
- moved ZD_PORT4 0.25 mm to (77.9, 73.7)
Connections:
- C_VCC pad 2: Net-(U1-SCL) -> Net-(U1-VCC)
- J1 pad 3: unconnected-(J1-Pin_3-Pad3) -> +3.3V
- R_EN pad 1: Net-(U1-SCL) -> Net-(U1-VCC)
- U1 pad 10: DGND -> SDA
- U1 pad 11: DGND -> SDA
- U1 pad 20: Net-(U1-SCL) -> Net-(U1-VCC)
- U1 pad 33: DGND -> (no net)
- U1 pad 6: unconnected-(U1-AUTO-Pad6) -> DGND
- U1 pad 9: Net-(U1-SCL) -> SCL
Routing:
- net +3.3V: track 0.00 -> 102.7 mm, vias 0 -> 1
- net DGND: track 36.5 -> 123.7 mm
- net Net-(U2-IO9): track 0.00 -> 39.0 mm, vias 0 -> 2
- net SDA: track 0.00 -> 23.0 mm, vias 0 -> 2
- net SCL: track 0.00 -> 22.8 mm, vias 0 -> 2
- net USB_D-: track 0.00 -> 21.0 mm
- net USB_D+: track 0.00 -> 18.3 mm
- net Net-(U1-SCL): track 17.5 -> 0.00 mm
- net Net-(U1-VCC): track 0.00 -> 14.3 mm
- net Net-(U2-EN): track 0.00 -> 8.97 mm, vias 0 -> 2
- net Net-(J2-CC2): track 0.00 -> 2.18 mm
- net Net-(J2-CC1): track 0.00 -> 2.17 mm
- net Net-(U1-PMAX): track 8.01 -> 8.82 mm
Other:
- board size 69.8 x 54.6 mm -> 74.9 x 54.6 mm
- board text added: "4-Port PSE v2.0"
- board text removed: "4-Port PSE v1.0"
